Commit message: Modification: disable collision model for "top_plate"

File: husky_description/urdf/decorations.urdf.xacro (robot description, xacro)
@@ -107,10 +107,10 @@
             </geometry>
           </visual>
-          <collision>
+          <!-- <collision>
             <origin xyz="0 0 0" rpy="0 0 0"/>
             <geometry>
               <mesh filename="package://husky_description/meshes/large_top_plate_collision.stl" />
             </geometry>
-          </collision>
+          </collision> -->
         </link>
         <!-- Attach top plate -->
@@ -141,10 +141,10 @@
             </geometry>
           </visual>
-          <collision>
+          <!-- <collision>
             <origin xyz="0 0 0" rpy="0 0 0"/>
             <geometry>
               <mesh filename="package://husky_description/meshes/top_plate.stl" />
             </geometry>
-          </collision>
+          </collision> -->
         </link>
         <!-- Attach top plate -->
