Commit message: ADD: dummy wheels for as_two_wheels

File: husky_description/urdf/husky_macro.urdf.xacro (robot description, xacro)
@@ -16,9 +16,10 @@
   <xacro:include filename="$(find husky_description)/urdf/decorations.urdf.xacro" />
   <xacro:include filename="$(find husky_description)/urdf/wheel.urdf.xacro" />
+  <xacro:include filename="$(find husky_description)/urdf/wheel_dummy.urdf.xacro" />
   <xacro:include filename="$(find husky_description)/urdf/accessories/intel_realsense.urdf.xacro"/>
   <!-- <xacro:include filename="$(find husky_description)/urdf/accessories/sick_lms1xx_mount.urdf.xacro"/> -->
   <xacro:include filename="$(find husky_description)/urdf/accessories/sensor_arch.urdf.xacro"/>
   <xacro:property name="M_PI" value="3.14159"/>
-  <xacro:macro name="husky" params="prefix">
+  <xacro:macro name="husky" params="prefix as_two_wheels:=false">
     <!-- Base Size -->
     <xacro:property name="base_x_size" value="0.98740000" />
@@ -89,17 +90,49 @@
       <child link="${prefix}gps_link" />
     </joint>
-    <!-- Husky wheel macros -->
-    <xacro:husky_wheel wheel_prefix="${prefix}front_left">
-      <origin xyz="${wheelbase/2} ${track/2} ${wheel_vertical_offset}" rpy="0 0 0" />
-    </xacro:husky_wheel>
-    <xacro:husky_wheel wheel_prefix="${prefix}front_right">
-      <origin xyz="${wheelbase/2} ${-track/2} ${wheel_vertical_offset}" rpy="0 0 0" />
-    </xacro:husky_wheel>
-    <xacro:husky_wheel wheel_prefix="${prefix}rear_left">
-      <origin xyz="${-wheelbase/2} ${track/2} ${wheel_vertical_offset}" rpy="0 0 0" />
-    </xacro:husky_wheel>
-    <xacro:husky_wheel wheel_prefix="${prefix}rear_right">
-      <origin xyz="${-wheelbase/2} ${-track/2} ${wheel_vertical_offset}" rpy="0 0 0" />
-    </xacro:husky_wheel>
+    <xacro:if value="$(arg as_two_wheels)">
+        <xacro:husky_wheel_dummy wheel_prefix="${prefix}front_left">
+            <origin xyz="${wheelbase/2} ${track/2} ${wheel_vertical_offset}" rpy="0 0 0" />
+        </xacro:husky_wheel_dummy>
+        <xacro:husky_wheel_dummy wheel_prefix="${prefix}front_right">
+            <origin xyz="${wheelbase/2} ${-track/2} ${wheel_vertical_offset}" rpy="0 0 0" />
+        </xacro:husky_wheel_dummy>
+        <xacro:husky_wheel_dummy wheel_prefix="${prefix}rear_left">
+            <origin xyz="${-wheelbase/2} ${track/2} ${wheel_vertical_offset}" rpy="0 0 0" />
+        </xacro:husky_wheel_dummy>
+        <xacro:husky_wheel_dummy wheel_prefix="${prefix}rear_right">
+            <origin xyz="${-wheelbase/2} ${-track/2} ${wheel_vertical_offset}" rpy="0 0 0" />
+        </xacro:husky_wheel_dummy>
+        <link name="${prefix}left_wheel"/>
+        <joint name="${prefix}left_wheel_joint" type="revolute">
+            <parent link="base_link"/>
+            <child link="${prefix}left_wheel"/>
+            <origin xyz="0 ${track/2} ${wheel_vertical_offset}" rpy="0 0 0" />
+            <axis rpy="0 0 0" xyz="0 1 0"/>
+            <limit effort="100.0" lower="-3.141592" upper="3.141592" velocity="1000"/>
+        </joint>
+        <link name="${prefix}right_wheel"/>
+        <joint name="${prefix}right_wheel_joint" type="revolute">
+            <parent link="base_link"/>
+            <child link="${prefix}right_wheel"/>
+            <origin xyz="0 ${-track/2} ${wheel_vertical_offset}" rpy="0 0 0" />
+            <axis rpy="0 0 0" xyz="0 1 0"/>
+            <limit effort="100.0" lower="-3.141592" upper="3.141592" velocity="1000"/>
+        </joint>
+    </xacro:if>
+    <xacro:unless value="$(arg as_two_wheels)">
+        <!-- Husky wheel macros -->
+        <xacro:husky_wheel wheel_prefix="${prefix}front_left">
+            <origin xyz="${wheelbase/2} ${track/2} ${wheel_vertical_offset}" rpy="0 0 0" />
+        </xacro:husky_wheel>
+        <xacro:husky_wheel wheel_prefix="${prefix}front_right">
+            <origin xyz="${wheelbase/2} ${-track/2} ${wheel_vertical_offset}" rpy="0 0 0" />
+        </xacro:husky_wheel>
+        <xacro:husky_wheel wheel_prefix="${prefix}rear_left">
+            <origin xyz="${-wheelbase/2} ${track/2} ${wheel_vertical_offset}" rpy="0 0 0" />
+        </xacro:husky_wheel>
+        <xacro:husky_wheel wheel_prefix="${prefix}rear_right">
+            <origin xyz="${-wheelbase/2} ${-track/2} ${wheel_vertical_offset}" rpy="0 0 0" />
+        </xacro:husky_wheel>
+    </xacro:unless>
     <xacro:husky_decorate />
     <!-- <xacro:if value="$(arg laser_enabled)">
@@ -133,54 +166,56 @@
       <xacro:intel_realsense_mount prefix="camera" topic="realsense" parent_link="realsense_mountpoint"/>
     </xacro:if>
-    <ros2_control name="${prefix}husky_hardware" type="system">
-      <hardware>
-        <xacro:if value="$(arg is_sim)">
-          <plugin>gazebo_ros2_control/GazeboSystem</plugin>
-        </xacro:if>
-        <xacro:unless value="$(arg is_sim)">
-          <plugin>husky_base/HuskyHardware</plugin>
-          <plugin>fake_components/GenericSystem</plugin>
-          <param name="hw_start_duration_sec">2.0</param>
-          <param name="hw_stop_duration_sec">3.0</param>
-          <param name="wheel_diameter">0.3302</param>
-          <param name="max_accel">5.0</param>
-          <param name="max_speed">1.0</param>
-          <param name="polling_timeout">10.0</param>
-          <param name="serial_port">/dev/ttyUSB0</param>
-        </xacro:unless>
-      </hardware>
-      <joint name="${prefix}front_left_wheel_joint">
-        <command_interface name="velocity">
-          <param name="min">-1</param>
-          <param name="max">1</param>
-        </command_interface>
-        <state_interface name="position"/>
-        <state_interface name="velocity"/>
-      </joint>
-      <joint name="${prefix}rear_left_wheel_joint">
-        <command_interface name="velocity">
-          <param name="min">-1</param>
-          <param name="max">1</param>
-        </command_interface>
-        <state_interface name="position"/>
-        <state_interface name="velocity"/>
-      </joint>
-      <joint name="${prefix}front_right_wheel_joint">
-        <command_interface name="velocity">
-          <param name="min">-1</param>
-          <param name="max">1</param>
-        </command_interface>
-        <state_interface name="position"/>
-        <state_interface name="velocity"/>
-      </joint>
-      <joint name="${prefix}rear_right_wheel_joint">
-        <command_interface name="velocity">
-          <param name="min">-1</param>
-          <param name="max">1</param>
-        </command_interface>
-        <state_interface name="position"/>
-        <state_interface name="velocity"/>
-      </joint>
-    </ros2_control>
+    <xacro:unless value="$(arg as_two_wheels)">
+        <ros2_control name="${prefix}husky_hardware" type="system">
+          <hardware>
+            <xacro:if value="$(arg is_sim)">
+              <plugin>gazebo_ros2_control/GazeboSystem</plugin>
+            </xacro:if>
+            <xacro:unless value="$(arg is_sim)">
+              <plugin>husky_base/HuskyHardware</plugin>
+              <plugin>fake_components/GenericSystem</plugin>
+              <param name="hw_start_duration_sec">2.0</param>
+              <param name="hw_stop_duration_sec">3.0</param>
+              <param name="wheel_diameter">0.3302</param>
+              <param name="max_accel">5.0</param>
+              <param name="max_speed">1.0</param>
+              <param name="polling_timeout">10.0</param>
+              <param name="serial_port">/dev/ttyUSB0</param>
+            </xacro:unless>
+          </hardware>
+          <joint name="${prefix}front_left_wheel_joint">
+            <command_interface name="velocity">
+              <param name="min">-1</param>
+              <param name="max">1</param>
+            </command_interface>
+            <state_interface name="position"/>
+            <state_interface name="velocity"/>
+          </joint>
+          <joint name="${prefix}rear_left_wheel_joint">
+            <command_interface name="velocity">
+              <param name="min">-1</param>
+              <param name="max">1</param>
+            </command_interface>
+            <state_interface name="position"/>
+            <state_interface name="velocity"/>
+          </joint>
+          <joint name="${prefix}front_right_wheel_joint">
+            <command_interface name="velocity">
+              <param name="min">-1</param>
+              <param name="max">1</param>
+            </command_interface>
+            <state_interface name="position"/>
+            <state_interface name="velocity"/>
+          </joint>
+          <joint name="${prefix}rear_right_wheel_joint">
+            <command_interface name="velocity">
+              <param name="min">-1</param>
+              <param name="max">1</param>
+            </command_interface>
+            <state_interface name="position"/>
+            <state_interface name="velocity"/>
+          </joint>
+        </ros2_control>
+    </xacro:unless>
   </xacro:macro>
 </robot>

Commit message: feat: add base_wheel_collision_box_link for collision model

File: husky_description/urdf/husky_macro.urdf.xacro (robot description, xacro)
@@ -34,4 +34,14 @@
     <xacro:property name="wheel_length" value="0.1143" />
     <xacro:property name="wheel_radius" value="0.1651" />
+    <!-- Aggregate collision box covering the base and all wheels -->
+    <xacro:property name="base_wheel_collision_x_min" value="${min(-(base_x_size / 2.0 + husky_rear_bumper_extend), -(wheelbase / 2.0 + wheel_radius))}" />
+    <xacro:property name="base_wheel_collision_x_max" value="${max(base_x_size / 2.0 + husky_front_bumper_extend, wheelbase / 2.0 + wheel_radius)}" />
+    <xacro:property name="base_wheel_collision_y_size" value="${2.0 * max(base_y_size / 2.0, track / 2.0 + wheel_length / 2.0)}" />
+    <xacro:property name="base_wheel_collision_z_min" value="${min(0.0, wheel_vertical_offset - wheel_radius)}" />
+    <xacro:property name="base_wheel_collision_z_max" value="${max(base_z_size, wheel_vertical_offset + wheel_radius)}" />
+    <xacro:property name="base_wheel_collision_x_size" value="${base_wheel_collision_x_max - base_wheel_collision_x_min}" />
+    <xacro:property name="base_wheel_collision_z_size" value="${base_wheel_collision_z_max - base_wheel_collision_z_min}" />
+    <xacro:property name="base_wheel_collision_x_origin" value="${(base_wheel_collision_x_max + base_wheel_collision_x_min) / 2.0}" />
+    <xacro:property name="base_wheel_collision_z_origin" value="${(base_wheel_collision_z_max + base_wheel_collision_z_min) / 2.0}" />
     <!-- Base link is the center of the robot's bottom plate -->
     <link name="${prefix}base_link">
@@ -55,4 +65,17 @@
       </collision>
     </link>
+    <link name="${prefix}base_wheel_collision_box_link">
+      <collision>
+        <origin xyz="0 0 0" rpy="0 0 0" />
+        <geometry>
+          <box size="${base_wheel_collision_x_size} ${base_wheel_collision_y_size} ${base_wheel_collision_z_size}" />
+        </geometry>
+      </collision>
+    </link>
+    <joint name="${prefix}base_wheel_collision_box_joint" type="fixed">
+      <origin xyz="${base_wheel_collision_x_origin} 0 ${base_wheel_collision_z_origin}" rpy="0 0 0" />
+      <parent link="${prefix}base_link" />
+      <child link="${prefix}base_wheel_collision_box_link" />
+    </joint>
     <!-- Base footprint is on the ground under the robot -->
     <link name="${prefix}base_footprint"/>
