Commit message: add:  "additional_comp" to xacro

File: husky_description/mjcf/husky_macro.xml.xacro (robot description, xacro)
@@ -19,5 +19,5 @@
   <xacro:include filename="$(find husky_description)/mjcf/wheel.xml.xacro" />
   <xacro:include filename="$(find husky_description)/mjcf/wheel_dummy.xml.xacro" />
-    <xacro:macro name="husky" params="prefix as_two_wheels:=false">
+    <xacro:macro name="husky" params="prefix:='' as_two_wheels:=false **additional_comp">
         <body name="${prefix}base_link" pos="0 0 ${wheel_radius - wheel_vertical_offset}">
             <inertial pos="-0.00065 -0.085 0.062"  mass="46.034" fullinertia="0.6022 1.7386 2.0296 -0.02364 -0.1197 -0.001544"/>
@@ -28,5 +28,6 @@
                 <inertial mass="0.001" pos="0 0 0" diaginertia="1e-6 1e-6 1e-6"/>
             </body>
-            <xacro:if value="$(arg as_two_wheels)">
+            <xacro:insert_block name="additional_comp" />
+            <xacro:if value="${as_two_wheels}">
                 <xacro:husky_wheel_dummy wheel_prefix="${prefix}front_left"
                                          xyz="${wheelbase/2.0} ${track/2.0} ${wheel_vertical_offset}" rpy="0 0 0"/>

File: husky_description/mjcf/husky_scene.xml.xacro (robot description, xacro)
@@ -5,5 +5,5 @@
     <xacro:include filename="$(find husky_description)/mjcf/husky_macro.xml.xacro" />
     <xacro:include filename="$(find husky_description)/mjcf/wheel_actuator.xml.xacro" />
-    <compiler angle="radian" meshdir="assets"/>
+    <compiler angle="radian" />
     <option timestep="0.001" integrator="implicit"/>
     <statistic center="0.2 0 0.4" extent=".8"/>
@@ -48,5 +48,7 @@
             <joint name="world_joint" type="free" stiffness="0" damping="0" frictionloss="0" armature="0" />
             <xacro:husky prefix="$(arg prefix)"
-                         as_two_wheels="$(arg as_two_wheels)"/>
+                         as_two_wheels="$(arg as_two_wheels)">
+                <additional_comp/>
+            </xacro:husky>
         </body>
     </worldbody>

Commit message: seperate assets & add imu

File: husky_description/mjcf/husky_macro.xml.xacro (robot description, xacro)
@@ -25,4 +25,5 @@
             <geom class="collision" size="${( base_x_size + husky_front_bumper_extend + husky_rear_bumper_extend)/2 } ${base_y_size/2} ${base_z_size/2/2}" pos="${( husky_front_bumper_extend - husky_rear_bumper_extend ) / 2.0} 0 ${base_z_size/4}" type="box"/>
             <geom class="collision" size="${base_x_size*4/5/2} ${base_y_size/2} ${(base_z_size/2-0.02)/2}" pos="0 0 ${base_z_size*3/4-0.01}" type="box"/>
+            <site name="${prefix}imu" size="0.01" pos="0 0 0" />
             <body name="${prefix}base_footprint" pos="0 0 ${wheel_vertical_offset - wheel_radius}">
                 <inertial mass="0.001" pos="0 0 0" diaginertia="1e-6 1e-6 1e-6"/>

File: husky_description/mjcf/husky_scene.xml.xacro (robot description, xacro)
@@ -5,4 +5,6 @@
     <xacro:include filename="$(find husky_description)/mjcf/husky_macro.xml.xacro" />
     <xacro:include filename="$(find husky_description)/mjcf/wheel_actuator.xml.xacro" />
+    <xacro:include filename="$(find husky_description)/mjcf/sensors.xml.xacro" />
+    <xacro:include filename="$(find husky_description)/mjcf/assets.xml.xacro" />
     <compiler angle="radian" />
     <option timestep="0.001" integrator="implicit"/>
@@ -32,13 +34,5 @@
         <texture type="2d" name="groundplane" builtin="checker" mark="edge" rgb1="0.2 0.3 0.4" rgb2="0.1 0.2 0.3" markrgb="0.8 0.8 0.8" width="300" height="300"/>
         <material name="groundplane" texture="groundplane" texuniform="true" texrepeat="5 5" reflectance="0.2"/>
-        <material class="husky" name="husky_orange" rgba="0.996 0.941 0.412 1.0"/>
-        <material class="husky" name="husky_black"  rgba="0.231 0.231 0.231 1.0"/>
-        <mesh name="base_link"       file="$(find husky_description)/meshes/base_link.stl"/>
-        <mesh name="wheel"           file="$(find husky_description)/meshes/wheel.stl"/>
-        <mesh name="bumper"          file="$(find husky_description)/meshes/bumper.obj"/>
-        <mesh name="top_chassis"     file="$(find husky_description)/meshes/top_chassis.stl"/>
-        <mesh name="top_plate"       file="$(find husky_description)/meshes/top_plate.stl"/>
-        <mesh name="large_top_plate" file="$(find husky_description)/meshes/large_top_plate.obj"/>
-        <mesh name="user_rail"       file="$(find husky_description)/meshes/user_rail.stl"/>
+        <xacro:husky_assets/>
     </asset>
     <worldbody>
@@ -55,3 +49,4 @@
     <xacro:husky_wheel_actuator prefix="$(arg prefix)"
                                 as_two_wheels="$(arg as_two_wheels)"/>
+    <xacro:husky_sensors prefix="$(arg prefix)"/>
 </mujoco>
